Commit message: chore: removed unuseful pkgs and updated docs

File: my_cart/urdf/my_robot.xacro (robot description, xacro)
@@ -128,18 +128,18 @@
     <pose>0 0 ${wheel_radius} 0 0 0</pose>
     <inertial>
-      <mass value="15.0"/>
+      <mass value="8.0"/>
       <origin xyz="0.0 0 0" rpy=" 0 0 0"/>
       <inertia
           ixx="0.1" ixy="0" ixz="0"
           iyy="0.1" iyz="0"
-          izz="0.1"
-      />
-    </inertial>
-    <collision name='chassis_collision'>
+          izz="0.001"
+      />
+    </inertial>
+    <!--collision name='chassis_collision'>
       <origin xyz="0 0 0" rpy=" 0 0 0"/>
       <geometry>
         <box size="${footprint_length} ${footprint_width} ${footprint_height}"/>
       </geometry>
-    </collision>
+    </collision-->
     <visual name='chassis_visual'>
       <origin xyz="0 0 0" rpy=" 0 0 0"/>
@@ -181,10 +181,10 @@
     </visual>
     <inertial>
-      <mass value="5.0"/>
+      <mass value="1.0"/>
       <origin xyz="0.0 0 0" rpy="0 1.5707 1.5707"/>
       <inertia
-          ixx="0.1" ixy="0" ixz="0"
-          iyy="0.1" iyz="0"
-          izz="0.1"
+          ixx="0.001" ixy="0" ixz="0"
+          iyy="0.001" iyz="0"
+          izz="0.005"
       />
     </inertial>
@@ -210,10 +210,10 @@
     </visual>
     <inertial>
-      <mass value="5.0"/>
+      <mass value="1.0"/>
       <origin xyz="0.0 0 0" rpy="0 1.5707 1.5707"/>
       <inertia
-          ixx="0.1" ixy="0" ixz="0"
-          iyy="0.1" iyz="0"
-          izz="0.1"
+          ixx="0.001" ixy="0" ixz="0"
+          iyy="0.001" iyz="0"
+          izz="0.005"
       />
     </inertial>
@@ -239,10 +239,10 @@
     </visual>
     <inertial>
-      <mass value="5.0"/>
+      <mass value="1.0"/>
       <origin xyz="0.0 0 0" rpy="0 1.5707 1.5707"/>
       <inertia
-          ixx="0.1" ixy="0" ixz="0"
-          iyy="0.1" iyz="0"
-          izz="0.1"
+          ixx="0.001" ixy="0" ixz="0"
+          iyy="0.001" iyz="0"
+          izz="0.005"
       />
     </inertial>
@@ -268,10 +268,10 @@
     </visual>
     <inertial>
-      <mass value="5.0"/>
+      <mass value="1.0"/>
       <origin xyz="0.0 0 0" rpy="0 1.5707 1.5707"/>
       <inertia
-          ixx="0.1" ixy="0" ixz="0"
-          iyy="0.1" iyz="0"
-          izz="0.1"
+          ixx="0.001" ixy="0" ixz="0"
+          iyy="0.001" iyz="0"
+          izz="0.005"
       />
     </inertial>
@@ -282,5 +282,5 @@
     <parent link="chassis"/>
     <axis xyz="0 1 0" rpy="0 0 0"/>
-    <limit effort="10000" velocity="1000"/>
+    <limit effort="40" velocity="100"/>
     <dynamics damping="1.0" friction="1.0"/>
   </joint>
@@ -290,5 +290,5 @@
     <parent link="chassis"/>
     <axis xyz="0 1 0" rpy="0 0 0"/>
-    <limit effort="10000" velocity="1000"/>
+    <limit effort="40" velocity="100"/>
     <dynamics damping="1.0" friction="1.0"/>
   </joint>
@@ -298,5 +298,5 @@
     <parent link="chassis"/>
     <axis xyz="0 1 0" rpy="0 0 0"/>
-    <limit effort="10000" velocity="1000"/>
+    <limit effort="40" velocity="100"/>
     <dynamics damping="1.0" friction="1.0"/>
   </joint>
@@ -306,15 +306,15 @@
     <parent link="chassis"/>
     <axis xyz="0 1 0" rpy="0 0 0"/>
-    <limit effort="10000" velocity="1000"/>
+    <limit effort="40" velocity="100"/>
     <dynamics damping="1.0" friction="1.0"/>
   </joint>
   <!-- ******* FRONT CAMERA ******* -->
   <link name="camera">
-    <collision name='camera_collision'>
+    <!--collision name='camera_collision'>
       <origin xyz="-${footprint_width/8} 0 0" rpy=" 0 1.57 0"/>
       <geometry>
         <cylinder radius="${footprint_width/10}" length="${footprint_width/4}"/>
       </geometry>
-    </collision>
+    </collision-->
     <visual name='camera_visual'>
       <origin xyz="-${footprint_width/8} 0 0" rpy=" 0 1.57 0"/>
@@ -342,14 +342,14 @@
   <!-- ******* LIDAR ******* -->
   <link name="hokuyo">
-    <collision name='hokuyo_collision'>
+    <!--collision name='hokuyo_collision'>
       <origin xyz="0 0 0" rpy="0 0 0"/>
       <geometry>
         <box size="0.1 0.1 0.1"/>
       </geometry>
-    </collision>
+    </collision-->
     <visual name='hokuyo_visual'>
       <origin xyz="0 0 0" rpy="0 0 0"/>
       <geometry>
-        <mesh filename="package://my_robot/meshes/hokuyo.dae"/>
+        <mesh filename="package://my_cart/meshes/hokuyo.dae"/>
       </geometry>
     </visual>

Commit message: feat: add kinect camera

File: my_cart/urdf/my_robot.xacro (robot description, xacro)
@@ -6,4 +6,5 @@
   <xacro:property name="footprint_height"  value="0.1" />
   <xacro:property name="footprint_length" value="0.5" />
+    <xacro:property name="M_PI" value="3.14159265359" />
   <xacro:include filename="$(find my_cart)/urdf/my_robot.gazebo" />
   <link name="robot_footprint"></link>
@@ -310,5 +311,5 @@
   </joint>
   <!-- ******* FRONT CAMERA ******* -->
-  <link name="camera">
+  <link name="camera_link">
     <!--collision name='camera_collision'>
       <origin xyz="-${footprint_width/8} 0 0" rpy=" 0 1.57 0"/>
@@ -335,8 +336,15 @@
   <joint type="fixed" name="camera_joint">
     <origin xyz="${footprint_width/4} 0 ${2*wheel_radius + 2*footprint_width/8}" rpy="0 0.10 0"/>
-    <child link="camera"/>
+    <child link="camera_link"/>
     <parent link="chassis"/>
     <axis xyz="0 1 0" rpy="0 0 0"/>
   </joint>
+  <joint name="camera_optical_joint" type="fixed">
+    <origin xyz="0 0 0" rpy="-1.5707 0 -1.5707"/>
+    <parent link="camera_link"/>
+    <child link="camera_link_optical"/>
+  </joint>
+  <link name="camera_link_optical">
+  </link>
   <!-- ******* -->
   <!-- ******* LIDAR ******* -->
@@ -392,5 +400,5 @@
     <material>Gazebo/Red</material>
 </gazebo>
-<gazebo reference="camera">
+<gazebo reference="camera_link">
     <material>Gazebo/Black</material>
 </gazebo>

Commit message: fix more feature in the appartment!

File: my_cart/urdf/my_robot.xacro (robot description, xacro)
@@ -283,5 +283,5 @@
     <parent link="chassis"/>
     <axis xyz="0 1 0" rpy="0 0 0"/>
-    <limit effort="40" velocity="100"/>
+    <limit effort="80" velocity="100"/>
     <dynamics damping="1.0" friction="1.0"/>
   </joint>
@@ -291,5 +291,5 @@
     <parent link="chassis"/>
     <axis xyz="0 1 0" rpy="0 0 0"/>
-    <limit effort="40" velocity="100"/>
+    <limit effort="80" velocity="100"/>
     <dynamics damping="1.0" friction="1.0"/>
   </joint>
@@ -299,5 +299,5 @@
     <parent link="chassis"/>
     <axis xyz="0 1 0" rpy="0 0 0"/>
-    <limit effort="40" velocity="100"/>
+    <limit effort="80" velocity="100"/>
     <dynamics damping="1.0" friction="1.0"/>
   </joint>
@@ -307,5 +307,5 @@
     <parent link="chassis"/>
     <axis xyz="0 1 0" rpy="0 0 0"/>
-    <limit effort="40" velocity="100"/>
+    <limit effort="80" velocity="100"/>
     <dynamics damping="1.0" friction="1.0"/>
   </joint>
